File: home.kicad_sch (KiCad schematic)
At the start: 49 parts, among them J1 OLED, J2 VS1838B IR Receiver, P1 USB_C_Plug_USB2.0, Q1 SS8050, SW1 SW_Push, SW2 SW_Push, U1 ESP32-S3-WROOM-1, U3 SCD41-D-R2, U4 BH1750FVI-TR, U5 AP2112K-3.3

Commit message: kiwi
Parts:
- renumbered D1 to D7, D7 to D8, D8 to D9
Changed lines of the file:
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@@
 		(dnp no)
 		(fields_autoplaced yes)
-		(property "Reference" "D1"
+		(property "Reference" "D7"
 			(at 82.55 27.6224 90)
 			(show_name no)
@@
 			(project "home"
 				(path "/d9bcb3ae-2a0c-45f9-9ce2-29d49931e58b"
-					(reference "D1")
+					(reference "D7")
 					(unit 1)
 				)
@@
 		(in_pos_files yes)
 		(dnp no)
-		(property "Reference" "D8"
+		(property "Reference" "D9"
 			(at 99.06 124.7774 90)
 			(show_name no)
@@
 			(project "home"
 				(path "/d9bcb3ae-2a0c-45f9-9ce2-29d49931e58b"
-					(reference "D8")
+					(reference "D9")
 					(unit 1)
 				)
@@
 		(in_pos_files yes)
 		(dnp no)
-		(property "Reference" "D7"
+		(property "Reference" "D8"
 			(at 67.31 124.968 90)
 			(show_name no)
@@
 			(project "home"
 				(path "/d9bcb3ae-2a0c-45f9-9ce2-29d49931e58b"
-					(reference "D7")
+					(reference "D8")
 					(unit 1)
 				)
