File: home.kicad_sch (KiCad schematic)
At the start: 49 parts, among them J1 OLED, J2 VS1838B IR Receiver, P1 USB_C_Plug_USB2.0, Q1 SS8050, SW1 SW_Push, SW2 SW_Push, U1 ESP32-S3-WROOM-1, U3 SCD41-D-R2, U4 BH1750FVI-TR, U5 AP2112K-3.3

Commit message: mondayWFH
Parts:
- removed C15: 100nF, Capacitor_SMD:C_0201_0603Metric, symbol Device:C_Small
- removed D1, D2: (no value), Diode_SMD:D_SOD-923, symbol Diode:ESD9B5.0ST5G
- removed D3, D4, D5, D6: WS2812B, LED_SMD:LED_WS2812B_PLCC4_5.0x5.0mm_P3.2mm, symbol LED:WS2812B
- removed D7: LED, LED_SMD:LED_0603_1608Metric, symbol Device:LED
- removed J1: OLED, Connector_PinHeader_1.00mm:PinHeader_1x04_P1.00mm_Vertical, symbol Connector:Conn_01x04_Pin
- removed P1: USB_C_Plug_USB2.0, symbol Connector:USB_C_Plug_USB2.0
- removed U1: ESP32-S3-WROOM-1, RF_Module:ESP32-S3-WROOM-1, symbol RF_Module:ESP32-S3-WROOM-1
- removed U5: AP2112K-3.3, Package_TO_SOT_SMD:SOT-23-5, symbol flumper:AP2112K-3.3
- added ANT1: 50Ohm 2.4GHz PCB ANT, parts:2.4GHz Antenna, symbol 2.4GHzAntenna:Antenna
- added C10, C11, C12, C17, C20, C25, C8: 100nF, Capacitor_SMD:C_0201_0603Metric, symbol Device:C_Small
- added C22, C24: 3p3F, Capacitor_SMD:C_0201_0603Metric, symbol Device:C_Small
- added C23: 20pF, Capacitor_SMD:C_0201_0603Metric, symbol Device:C_Small
- added C4: 10uF, Capacitor_SMD:C_0201_0603Metric, symbol Device:C_Small
- added C9: 1uF, Capacitor_SMD:C_0201_0603Metric, symbol Device:C_Small
- added D1: LED, LED_SMD:LED_0603_1608Metric, symbol Device:LED
- added J1: USB_C_Receptacle_USB2.0_14P, Connector_USB:USB_C_Receptacle_GCT_USB4105-xx-A_16P_TopMnt_Horizontal, symbol Connector:USB_C_Receptacle_USB2.0_14P
- added J2: JST, Connector_PinHeader_2.54mm:PinHeader_1x04_P2.54mm_Vertical, symbol Connector:Conn_01x04_Socket
- added J3: DISPLAY, parts:LCSC FPC 18, symbol Connector:Conn_01x18_Socket
- added J4: Micro_SD_Card, parts:MicroSD LCSC, symbol Connector:Micro_SD_Card
- added L1, L2, L3: 2n2H, Inductor_SMD:L_0201_0603Metric, symbol Device:L_Small
- added R10, R14, R15, R16, R17, R19: 10k, Resistor_SMD:R_0201_0603Metric, symbol Device:R
- added R13: 22R, Resistor_SMD:R_0201_0603Metric, symbol Device:R
- added R2: 1M, Resistor_SMD:R_0201_0603Metric, symbol Device:R
- added R5: 5.1k, Resistor_SMD:R_0201_0603Metric, symbol Device:R
- added R9: 47R, Resistor_SMD:R_0201_0603Metric, symbol Device:R
- added U1: USBLC6-2SC6, Package_TO_SOT_SMD:SOT-23-6, symbol Power_Protection:USBLC6-2SC6
- added U2: ESP32-S3, Package_DFN_QFN:QFN-56-1EP_7x7mm_P0.4mm_EP4x4mm, symbol MCU_Espressif:ESP32-S3
- added U3: SPX3819M5-L-3-3, Package_TO_SOT_SMD:SOT-23-5, symbol flumper:SPX3819M5-L-3-3
- added U4: ESP-PSRAM64H, Package_SO:SOIC-8_3.9x4.9mm_P1.27mm, symbol Memory_RAM:ESP-PSRAM32
- added U5: W25Q128JVSIQ, Package_SO:SOIC-8_5.3x5.3mm_P1.27mm, symbol Memory_Flash:W25Q128JVS
- added Y1: 40MHz, Crystal:Crystal_SMD_EuroQuartz_X22-4Pin_2.5x2.0mm, symbol Device:Crystal_GND24_Small
- C1: value 100uF -> 2.2nF
- C13, C5: value 100nF -> 1uF
- C16: value 100nF -> 10uF
- C19: value 10nF -> 20pF
- C2: value 2.2nF -> 1uF
- C21: renamed from C4; value 1uF -> 10uF
- C3: value 1uF -> 10nF
- C6: value 1uF -> 100nF
- C7: value 22uF -> 100nF
- D2: renamed from D8; footprint LED_SMD:LED_1206_3216Metric -> LED_THT:LED_D1.8mm_W1.8mm_H2.4mm_Horizontal_O3.81mm_Z1.6mm
- D3: renamed from D9; footprint LED_SMD:LED_1206_3216Metric -> LED_THT:LED_D1.8mm_W1.8mm_H2.4mm_Horizontal_O3.81mm_Z1.6mm
- J5: renamed from J2; footprint Connector_PinHeader_1.00mm:PinHeader_1x03_P1.00mm_Vertical -> Connector_PinSocket_2.54mm:PinSocket_1x03_P2.54mm_Vertical
- R1: value 2.2k -> 4.7kR
- R20: renamed from R9; value 220 -> 1k
- R3: value 1M -> 4.7kR
- R6: value 4.7k -> 2.2k
- R7: value 4.7k -> 10k
- R8: value 330 -> 470R
- SW1, SW2: footprint (none) -> Button_Switch_SMD:SW_SPST_PTS810
- U6: renamed from U4; footprint BH1750FVI-TR:XDCR_BH1750FVI-TR -> parts:XDCR_BH1750FVI-TR
- renumbered C8 to C15, C12 to C26, C9 to C27, C10 to C28, C17 to C29, C11 to C30, R4 to R11, R5 to R12, R10 to R18, R11 to R21, R2 to R4, U3 to U7
Connections:
- net BOOT: now also C17.1, U2.5 (GPIO0)
- net D+: now also U1.4 (I/O2), U2.26 (GPIO20/USB_D+)
- net D-: now also U1.6 (I/O1), U2.25 (GPIO19/USB_D-)
- net EN: now also J3.8 (Pin_8), U2.4 (CHIP_PU)
- net GND: now also C1.1, C18.1, C2.2, C3.2, R4.1, ANT1.2 (GND), C10.1, C11.1, C12.1, C17.2, C20.1, C22.1, C23.1, C24.1, C25.1, C4.1, C8.1, C9.1, D1.1 (K), J1.A1 (GND), J1.A12 (GND), J1.B1 (GND), J1.B12 (GND), J2.2 (Pin_2), J3.10 (Pin_10), J3.11 (Pin_11), J3.16 (Pin_16), J3.17 (Pin_17), J3.18 (Pin_18), J3.3 (Pin_3), J3.6 (Pin_6), J4.6 (VSS), J4.SH (SHIELD), R2.1, R5.1, U1.2 (GND), U2.57 (GND), U3.2 (GND), U4.4 (VSS), U5.4 (GND), Y1.2 (G), Y1.4 (G); no longer C1.2, C18.2, C2.1, C3.1, R3.1, R4.2
- net IR-IN: now also U2.11 (GPIO6)
- net IR-OUT: now also U2.12 (GPIO7)
- net SCL: now also R3.1, J3.13 (Pin_13), U2.24 (GPIO18); no longer R7.1
- net SDA: now also R1.1, J3.14 (Pin_14), U2.23 (GPIO17); no longer R6.1
- net VBUS: now also C14.2, C16.2, L2.2, U3.1 (IN), U3.3 (EN); no longer C1.1, C18.1, C19.1, C3.2, R1.1
- net 3V3: now reaches R3.2
- net 3V3: now also C2.1, C21.2, C27.2, C28.2, C29.2, C3.1, C30.2, C5.2, C6.2, J5.1 (Pin_1), R1.2, R11.2, R12.2, R7.2, U6.1 (VCC), U7.19 (VDD), U7.7 (VDD), C10.2, C11.2, C12.2, C4.2, C9.2, J2.4 (Pin_4), J3.1 (Pin_1), J4.4 (VDD), L1.2, R10.2, R14.2, R15.2, R16.2, R17.2, R19.2, U2.20 (VDD3P3_RTC), U2.46 (VDD3P3_CPU), U2.55 (VDDA), U2.56 (VDDA), U3.5 (OUT); no longer C2.2
- net TX: now reaches R8.1
- net TX: now also J2.1 (Pin_1)
- net LED: no longer names the net of R8.2
- net LED: now also U2.49 (U0TXD)
- removed net V3.3: C13.2, C14.2, C16.2, C21.2, C27.2, C28.2, C29.2, C30.2, C5.2, C6.2, C7.2, J5.1 (Pin_1), R11.2, R12.2, R6.2, R7.2, U6.1 (VCC), U7.19 (VDD), U7.7 (VDD)
- new net: R9.2, U2.41 (GPIO36)
- new net: C19.1, R13.1, Y1.1
- new net: ANT1.1 (LNA), C24.2, L3.2
- new net: C8.2, J1.A4 (VBUS), J1.A9 (VBUS), J1.B4 (VBUS), J1.B9 (VBUS), L2.1, R6.1, U1.5 (VBUS)
- new net: J1.A5 (CC1), R5.2
- new net: J1.A6 (D+), J1.B6 (D+), U1.3 (I/O2)
- new net: J1.A7 (D-), J1.B7 (D-), U1.1 (I/O1)
- new net: J1.B5 (CC2), R4.2
- new net: C1.2, J1.SH (SHIELD), R2.2
- new net: D1.2 (A), R6.2
- new net: C18.2, U3.4 (BP)
- new net: C7.2, L1.1, U2.2 (VDD3P3), U2.3 (VDD3P3)
- new net CLK: J4.5 (CLK), R9.1
- new net CMD: J4.3 (CMD), R16.1, U2.40 (GPIO35)
- new net DAT0: J4.7 (DAT0), R17.1, U2.42 (GPIO37)
- new net DAT1: J4.8 (DAT1), R19.1, U2.43 (GPIO38)
- new net DAT2: J4.1 (DAT2), R14.1, U2.38 (GPIO33)
- new net DAT3: J4.2 (DAT3/CD), R15.1, U2.39 (GPIO34)
- new net FSPICLK: J3.4 (Pin_4), U2.17 (GPIO12)
- new net FSPICS0: J3.9 (Pin_9), U2.15 (GPIO10)
- new net FSPID: J3.5 (Pin_5), U2.16 (GPIO11)
- new net IO1: U2.6 (GPIO1)
- new net IO2: U2.7 (GPIO2)
- new net IO21: U2.27 (GPIO21)
- new net IO3: U2.8 (GPIO3)
- new net IO4: U2.9 (GPIO4)
- new net IO45: U2.51 (GPIO45)
- new net IO46: U2.52 (GPIO46)
- new net IO5: U2.10 (GPIO5)
- new net LCD_BL: J3.2 (Pin_2), U2.13 (GPIO8)
- new net LCD_DC: J3.7 (Pin_7), U2.14 (GPIO9)
- new net LNA_IN: C22.2, L3.1, U2.1 (LNA_IN)
- new net RX: J2.3 (Pin_3), U2.50 (U0RXD)
- new net SPICLK: U2.33 (SPICLK), U4.6 (SCLK), U5.6 (CLK)
- new net SPICS0: R10.1, U2.32 (SPICS0), U5.1 (~{CS})
- new net SPICS1: R7.1, U2.28 (SPICS1), U4.1 (~{CE})
- new net SPID: U2.35 (SPID), U4.5 (SI/SIO), U5.5 (DI/IO_{0})
- new net SPIHD: U2.30 (SPIHD), U4.7 (SIO3), U5.7 (~{HOLD}/~{RESET}/IO_{3})
- new net SPIQ: U2.34 (SPIQ), U4.2 (SO/SIO), U5.2 (DO/IO_{1})
- new net SPIWP: U2.31 (SPIWP), U4.3 (SIO2), U5.3 (~{WP}/IO_{2})
- new net TP_INT: J3.15 (Pin_15), U2.19 (GPIO14)
- new net TP_RST: J3.12 (Pin_12), U2.18 (GPIO13)
- new net VCC_SPI: C13.2, C20.2, C25.2, U2.29 (VDD_SPI), U4.8 (VCC), U5.8 (VCC)
- new net XTAL_N: C23.2, U2.53 (XTAL_N), Y1.3
- new net XTAL_P: R13.2, U2.54 (XTAL_P)
- no-connect marks 4 -> 8
Other:
- note added: "-JTAG-"
- note added: "Antenna and impedance matching circuit"
- note added: "ESP32-S3"
- note added: "FSPIHD"
- note added: "FSPIQ (MISO)"
- note added: "FSPIWP"
- note added: "GND"
- note added: "I2C address = 0x15"
- note added: "I2C address = 0x23 (ADDR = Low) = 0x5C (ADDR = High)"
- note added: "I2C address = 0x62"
- note added: "LCD_BL"
- note added: "LCD_CS"
- note added: "LCD_DC"
- note added: "LCD_MOSI"
- note added: "LCD_RST"
- note added: "LCD_SCLK"
- note added: "Lazy Kiwi Smart Home Device"
- note added: "Peripherals"
- note added: "Quad SPI Flash 16MB & PSRAM 8MB"
- note added: "SD Card reader"
- note added: "Smart home ESP32 device Designed and built from scratch as a learning exercise by Jonathan Black"
- note added: "Strapping pin"
- note added: "TP_INT"
- note added: "TP_RST"
- note added: "TP_SCL"
- note added: "TP_SDA"
- note added: "Touch Screen"
- note added: "UART Breakout"
- note added: "UNUSED"
- note added: "VCC"
- note added: "XTAL"
- note removed: "Camera, motion,"
- note removed: "OLED Display"
- note removed: "Smart home ESP32 device Designed by Jonathan Black"
- note removed: "Status LED"
- note removed: "uF and nF DONT CONFUSE!"
- moved on the sheet: C15, C21, C26, C27, C28, C29, C30, D2, D3, J5, Q1, R11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

Commit message: mondayWFH
Parts:
- added R10, R11, R12, R8, R9: 0R, Resistor_SMD:R_0201_0603Metric, symbol Device:R
- renumbered R8 to R13, R9 to R14, R10 to R15, R11 to R16, R12 to R17, R13 to R18, R14 to R19, R15 to R20, R16 to R21, R17 to R22, R18 to R23, R19 to R24, R20 to R25, R21 to R26
Connections:
- net SPICLK: now also R10.1; no longer U2.33 (SPICLK)
- net SPID: now also R12.1; no longer U2.35 (SPID)
- net SPIHD: now also R8.1; no longer U2.30 (SPIHD)
- net SPIQ: now also R11.1; no longer U2.34 (SPIQ)
- net SPIWP: now also R9.1; no longer U2.31 (SPIWP)
- new net: R9.2, U2.31 (SPIWP)
- new net: R11.2, U2.34 (SPIQ)
- new net: R10.2, U2.33 (SPICLK)
- new net: R12.2, U2.35 (SPID)
- new net: R8.2, U2.30 (SPIHD)
Other:
- moved on the sheet: R15
