File: home.kicad_sch (KiCad schematic)
At the start: 87 parts, among them J1 USB_C_Receptacle_USB2.0_14P, J2 JST, J3 DISPLAY, J4 Micro_SD_Card, J5 VS1838B IR Receiver, Q1 SS8050, SW1 SW_Push, SW2 SW_Push, U1 USBLC6-2SC6, U2 ESP32-S3, U3 SPX3819M5-L-3-3, U4 ESP-PSRAM64H, U5 W25Q128JVSIQ, U6 BH1750FVI-TR, U7 SCD41-D-R2, Y1 40MHz

Commit message: Thurs
Parts:
- removed J2: JST, Connector_PinHeader_2.54mm:PinHeader_1x04_P2.54mm_Vertical, symbol Connector:Conn_01x04_Socket
- added 3V3, GND, RX, SCL, SDA, TX: TestPoint, TestPoint:TestPoint_Pad_D1.0mm, symbol Connector:TestPoint
- J4: footprint parts:MicroSD LCSC -> Connector_Card:microSD_HC_Molex_104031-0811
- renumbered TP1 to IO1, TP3 to IO2, TP5 to IO3, TP7 to IO4, TP2 to IO5, TP4 to IO6, TP6 to IO7, TP8 to IO8
Connections:
- net 3V3: now also 3V3.1
- net GND: now also GND.1
- net RX: now also RX.1
- net SCL: now also SCL.1
- net SDA: now also SDA.1
- net TX: now also TX.1
Other:
- note removed: "UART Breakout"

Commit message: sklfdjaj
Parts:
- added Alert1: TP, TestPoint:TestPoint_Pad_D1.0mm, symbol Connector:TestPoint
- added C26: 100n, Capacitor_SMD:C_0402_1005Metric, symbol Device:C_Small
- added U6: MCP9808_DFN, Package_DFN_QFN:DFN-8-1EP_3x2mm_P0.5mm_EP1.7x1.4mm, symbol Sensor_Temperature:MCP9808_DFN
- C1: value 2.2nF -> 2n2
- C10, C11, C12, C14, C15, C17, C18, C20, C25, C6, C7, C8: value 100nF -> 100n
- C13, C2, C5, C9: value 1uF -> 1u
- C16, C21, C4: value 10uF -> 10u
- C19, C23: value 20pF -> 20p
- C22, C24: value 3p3F -> 3p3
- C27: renamed from C26; value 1uF -> 1u
- C28: renamed from C27; value 1uF -> 1u
- C29: renamed from C28; value 100nF -> 100n
- C3: value 10nF -> 10n
- C30: renamed from C29; value 100nF -> 100n
- C31: renamed from C30; value 100nF -> 100n
- L1, L2, L3: value 2n2H -> 2n2
- R1, R3: value 4.7kR -> 5k1
- R13: value 470R -> 470
- R14: value 47R -> 47
- R18: value 22R -> 22
- R23, R26: footprint Resistor_SMD:R_0402_1005Metric -> Resistor_SMD:R_0805_2012Metric
- R4, R5: value 5.1k -> 5k1
- R6: value 2.2k -> 2k1
- renumbered 3V3 to 3V1, GND to GND1, J3 to J2, J4 to J3, J5 to J4, RX to RX1, SCL to SCL1, SDA to SDA1, TX to TX1, U6 to U7, U7 to U8
Connections:
- net 3V3: now also C26.2, U6.8 (V_{DD})
- net GND: now also C26.1, U6.4 (GND), U6.5 (A2), U6.6 (A1), U6.7 (A0), U6.9 (EP/GND)
- net SCL: now also U6.2 (SCL)
- net SDA: now also U6.1 (SDA)
- new net: Alert1.1, U6.3 (Alert)
Other:
- note added: "High power rated resistors! Hence larger package"
- note added: "I2C address = 0x18"
- note added: "Temp Sensor"
- moved on the sheet: 3V1, GND1, IO1, IO2, IO3, IO4, IO5, IO6, IO7, IO8, J3, R19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
