File: home.kicad_pcb (KiCad board)
At the start: 4 copper layers, 46 parts, among them J1 OLED, J2 VS1838B IR Receiver, Q1 SS8050, U1 ESP32-S3-WROOM-1, U3 SCD41-D-R2, U5 AP2112K-3.3

Commit message: mondayWFH
Parts:
- removed D4, D5, D6: WS2812B, LED_SMD:LED_WS2812B_PLCC4_5.0x5.0mm_P3.2mm
- removed D7: LED, LED_SMD:LED_0603_1608Metric
- removed D8, D9: 940nm, LED_SMD:LED_1206_3216Metric
- added ANT1: 50Ohm 2.4GHz PCB ANT, parts:2.4GHz Antenna, F.Cu at (96.5, 60.6)
- added C20: 100nF, Capacitor_SMD:C_0201_0603Metric, F.Cu at (119.2, 69.5)
- added C21: 10uF, Capacitor_SMD:C_0201_0603Metric, F.Cu at (121.6, 53.8)
- added C22: 3p3F, Capacitor_SMD:C_0201_0603Metric, F.Cu at (121.6, 55.5)
- added C23: 20pF, Capacitor_SMD:C_0201_0603Metric, F.Cu at (121.6, 57.2)
- added C24: 3p3F, Capacitor_SMD:C_0201_0603Metric, F.Cu at (121.6, 59.0)
- added C25: 100nF, Capacitor_SMD:C_0201_0603Metric, F.Cu at (121.6, 60.8)
- added C26: 1uF, Capacitor_SMD:C_0201_0603Metric, F.Cu at (121.6, 62.5)
- added C27: 1uF, Capacitor_SMD:C_0201_0603Metric, F.Cu at (121.6, 64.2)
- added C28: 100nF, Capacitor_SMD:C_0201_0603Metric, F.Cu at (121.6, 66.0)
- added C29: 100nF, Capacitor_SMD:C_0201_0603Metric, F.Cu at (121.6, 67.8)
- added C30: 100nF, Capacitor_SMD:C_0201_0603Metric, F.Cu at (121.6, 69.5)
- added J3: DISPLAY, parts:LCSC FPC 18, F.Cu at (111.5, 50.0)
- added J4: Micro_SD_Card, parts:MicroSD LCSC, F.Cu at (119.0, 78.8)
- added J5: VS1838B IR Receiver, Connector_PinSocket_2.54mm:PinSocket_1x03_P2.54mm_Vertical, F.Cu at (178.7, 116.8)
- added L1: 2n2H, Inductor_SMD:L_0201_0603Metric, F.Cu at (124.1, 53.8)
- added L2: 2n2H, Inductor_SMD:L_0201_0603Metric, F.Cu at (124.1, 55.5)
- added L3: 2n2H, Inductor_SMD:L_0201_0603Metric, F.Cu at (124.1, 57.2)
- added R12: 10k, Resistor_SMD:R_0201_0603Metric, F.Cu at (126.5, 60.8)
- added R13: 22R, Resistor_SMD:R_0201_0603Metric, F.Cu at (126.5, 62.5)
- added R14: 10k, Resistor_SMD:R_0201_0603Metric, F.Cu at (126.5, 64.2)
- added R15: 10k, Resistor_SMD:R_0201_0603Metric, F.Cu at (126.5, 66.0)
- added R16: 10k, Resistor_SMD:R_0201_0603Metric, F.Cu at (126.5, 67.8)
- added R17: 10k, Resistor_SMD:R_0201_0603Metric, F.Cu at (126.5, 69.5)
- added R18: 47, Resistor_SMD:R_0201_0603Metric, F.Cu at (129.0, 53.8)
- added R19: 10k, Resistor_SMD:R_0201_0603Metric, F.Cu at (129.0, 55.5)
- added R20: 1k, Resistor_SMD:R_0201_0603Metric, F.Cu at (129.0, 57.2)
- added R21: 47, Resistor_SMD:R_0201_0603Metric, F.Cu at (129.0, 59.0)
- added SW1: SW_Push, Button_Switch_SMD:SW_SPST_PTS810, F.Cu at (180.0, 100.3)
- added SW2: SW_Push, Button_Switch_SMD:SW_SPST_PTS810, F.Cu at (180.0, 105.0)
- added U2: ESP32-S3, Package_DFN_QFN:QFN-56-1EP_7x7mm_P0.4mm_EP4x4mm, F.Cu at (111.1, 65.0)
- added U4: ESP-PSRAM64H, Package_SO:SOIC-8_3.9x4.9mm_P1.27mm, F.Cu at (168.9, 120.9)
- added U6: BH1750FVI-TR, parts:XDCR_BH1750FVI-TR, F.Cu at (176.4, 80.1)
- added U7: SCD41-D-R2, Sensor:Sensirion_SCD4x-1EP_10.1x10.1mm_P1.25mm_EP4.8x4.8mm, F.Cu at (102.5, 75.3)
- added Y1: 40MHz, Crystal:Crystal_SMD_EuroQuartz_X22-4Pin_2.5x2.0mm, F.Cu at (181.1, 80.5)
- C1: value 100uF -> 2.2nF
- C12, C6: value 1uF -> 100nF
- C13, C5: value 100nF -> 1uF
- C16: value 100nF -> 10uF
- C19: value 10nF -> 20pF
- C2: value 2.2nF -> 1uF
- C3: value 1uF -> 10nF
- C4: value 1uF -> 10uF
- C7: value 22uF -> 100nF
- D1: value ~ -> LED; footprint Diode_SMD:D_SOD-923 -> LED_SMD:LED_0603_1608Metric
- D2: value ~ -> 940nm; footprint Diode_SMD:D_SOD-923 -> LED_THT:LED_D1.8mm_W1.8mm_H2.4mm_Horizontal_O3.81mm_Z1.6mm
- D3: value WS2812B -> 940nm; footprint LED_SMD:LED_WS2812B_PLCC4_5.0x5.0mm_P3.2mm -> LED_THT:LED_D1.8mm_W1.8mm_H2.4mm_Horizontal_O3.81mm_Z1.6mm
- G***: moved to B.Cu
- J1: value OLED -> USB_C_Receptacle_USB2.0_14P; footprint Connector_PinHeader_1.00mm:PinHeader_1x04_P1.00mm_Vertical -> Connector_USB:USB_C_Receptacle_GCT_USB4105-xx-A_16P_TopMnt_Horizontal
- J2: value VS1838B IR Receiver -> JST; footprint Connector_PinHeader_1.00mm:PinHeader_1x03_P1.00mm_Vertical -> Connector_PinHeader_2.54mm:PinHeader_1x04_P2.54mm_Vertical
- R1: value 2.2k -> 4.7kR
- R10, R11: value 47 -> 10k
- R2: value 5.1k -> 1M
- R3: value 1M -> 4.7kR
- R4, R5: value 10k -> 5.1k
- R6: value 4.7k -> 2.2k
- R7: value 4.7k -> 10k
- R8: value 330 -> 470R
- R9: value 220 -> 47R
- U1: value ESP32-S3-WROOM-1 -> USBLC6-2SC6; footprint RF_Module:ESP32-S3-WROOM-1 -> Package_TO_SOT_SMD:SOT-23-6
- U3: value SCD41-D-R2 -> SPX3819M5-L-3-3; footprint Sensor:Sensirion_SCD4x-1EP_10.1x10.1mm_P1.25mm_EP4.8x4.8mm -> Package_TO_SOT_SMD:SOT-23-5
- U5: value AP2112K-3.3 -> W25Q128JVSIQ; footprint Package_TO_SOT_SMD:SOT-23-5 -> Package_SO:SOIC-8_5.3x5.3mm_P1.27mm
- moved U3 100.5 mm to (186.0, 104.9)
- moved U1 95.6 mm to (186.0, 100.3)
- moved D1 77.6 mm to (180.9, 83.8)
- moved C11 72.1 mm to (119.2, 53.8)
- moved C12 72.1 mm to (119.2, 55.5)
- moved Q1 70.4 mm to (176.1, 83.9)
- moved D3 70.1 mm to (184.6, 87.9)
- moved R10 69.6 mm to (126.5, 57.2)
- moved R11 69.6 mm to (126.5, 59.0)
- moved R8 69.6 mm to (126.5, 53.8)
- moved R9 69.6 mm to (126.5, 55.5)
- moved C1 67.1 mm to (116.7, 53.8)
- moved C2 67.1 mm to (116.7, 55.5)
- moved C3 67.1 mm to (116.7, 57.2)
- moved C4 67.1 mm to (116.7, 59.0)
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Connections:
- C1 pad 1: VBUS -> GND
- C1 pad 2: GND -> Net-(J1-SHIELD)
- C10 pad 2: V3.3 -> 3V3
- C11 pad 2: V3.3 -> 3V3
- C12 pad 2: Net-(U4-DVI) -> 3V3
- C13 pad 2: V3.3 -> VCC_SPI
- C14 pad 2: V3.3 -> VBUS
- C15 pad 1: GND -> EN
- C15 pad 2: V3.3 -> GND
- C16 pad 2: V3.3 -> VBUS
- C17 pad 1: GND -> BOOT
- C17 pad 2: V3.3 -> GND
- C18 pad 1: VBUS -> GND
- C18 pad 2: GND -> Net-(U3-BP)
- C19 pad 1: VBUS -> Net-(C19-Pad1)
- C2 pad 1: GND -> 3V3
- C2 pad 2: Net-(P1-SHIELD) -> GND
- C3 pad 1: GND -> 3V3
- C3 pad 2: VBUS -> GND
- C4 pad 2: V3.3 -> 3V3
- C5 pad 2: V3.3 -> 3V3
- C6 pad 2: V3.3 -> 3V3
- C7 pad 2: V3.3 -> Net-(C7-Pad2)
- C8 pad 1: EN -> GND
- C8 pad 2: GND -> Net-(U1-VBUS)
- C9 pad 2: V3.3 -> 3V3
- D1 pad 2: D+ -> Net-(D1-A)
- D2 pad 1: GND -> Net-(D2-K)
- D2 pad 2: D- -> Net-(D2-A)
- D3 pad 1: V3.3 -> Net-(D2-K)
- J2 pad 1: V3.3 -> TX
- J2 pad 3: IR-IN -> RX
- Q1 pad 3: Net-(D8-K) -> Net-(D2-K)
- R1 pad 1: VBUS -> SDA
- R1 pad 2: Net-(D7-A) -> 3V3
- R10 pad 1: VBUS -> SPICS0
- R10 pad 2: Net-(D8-A) -> 3V3
- R11 pad 1: Net-(D9-A) -> EN
- R11 pad 2: VBUS -> 3V3
- R2 pad 1: Net-(P1-CC) -> GND
- R2 pad 2: GND -> Net-(J1-SHIELD)
- R3 pad 1: GND -> SCL
- R3 pad 2: Net-(P1-SHIELD) -> 3V3
- R4 pad 1: EN -> GND
- R4 pad 2: V3.3 -> Net-(J1-CC2)
- R5 pad 1: BOOT -> GND
- R5 pad 2: V3.3 -> Net-(J1-CC1)
- R6 pad 1: SDA -> Net-(U1-VBUS)
- R6 pad 2: V3.3 -> Net-(D1-A)
- R7 pad 1: SCL -> SPICS1
- R7 pad 2: V3.3 -> 3V3
- R8 pad 1: Net-(D3-DIN) -> TX
- R8 pad 2: LED -> Net-(U2-U0TXD)
- R9 pad 1: IR-OUT -> CLK
- R9 pad 2: Net-(Q1-B) -> Net-(U2-GPIO36)
- U1 pad 1: GND -> Net-(J1-D--PadA7)
- U1 pad 2: V3.3 -> GND
- U1 pad 3: EN -> Net-(J1-D+-PadA6)
- U1 pad 4: IR-IN -> D+
- U1 pad 5: IR-OUT -> Net-(U1-VBUS)
- U1 pad 6: unconnected-(U1-IO6-Pad6) -> D-
- U3 pad 1: (no net) -> VBUS
- U3 pad 2: (no net) -> GND
- U3 pad 3: (no net) -> VBUS
- U3 pad 4: (no net) -> Net-(U3-BP)
- U3 pad 5: (no net) -> 3V3
- U5 pad 1: VBUS -> SPICS0
- U5 pad 2: GND -> SPIQ
- U5 pad 3: VBUS -> SPIWP
- U5 pad 4: unconnected-(U5-NC-Pad4) -> GND
- U5 pad 5: V3.3 -> SPID
Other:
- board outline added: 35 x 42 mm

Commit message: mondayWFH
Parts:
- added R22: 10k, Resistor_SMD:R_0201_0603Metric, F.Cu at (107.5, 72.4)
- added R23: 47, Resistor_SMD:R_0201_0603Metric, F.Cu at (107.5, 74.1)
- added R24: 10k, Resistor_SMD:R_0201_0603Metric, F.Cu at (107.5, 75.9)
- added R25: 1k, Resistor_SMD:R_0201_0603Metric, F.Cu at (107.5, 77.6)
- added R26: 47, Resistor_SMD:R_0201_0603Metric, F.Cu at (107.5, 79.4)
- R10, R11, R12: value 10k -> 0R
- R13: value 22R -> 470R
- R14: value 10k -> 47R
- R18: value 47 -> 22R
- R20: value 1k -> 10k
- R21: value 47 -> 10k
- R8: value 470R -> 0R
- R9: value 47R -> 0R
- moved U1 90.8 mm to (96.6, 84.4)
- moved U3 90.8 mm to (96.6, 89.0)
- moved Y1 80.1 mm to (101.4, 88.5)
- moved J5 77.2 mm to (134.8, 53.3)
- moved D1 75.3 mm to (105.7, 87.7)
- moved Q1 74.5 mm to (101.6, 84.2)
- moved U4 64.2 mm to (112.9, 89.6)
- moved J2 60.4 mm to (130.2, 53.3), turned to 0 degrees
- moved D3 60.0 mm to (128.6, 66.2)
- moved SW1 48.9 mm to (133.4, 85.6)
- moved SW2 48.9 mm to (133.4, 90.3)
- moved U6 43.0 mm to (133.5, 77.8)
- moved D2 36.7 mm to (122.6, 66.2)
- moved J3 34.9 mm to (144.7, 60.6)
- moved U2 32.7 mm to (80.7, 77.1), turned to 180 degrees
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Connections:
- R10 pad 1: SPICS0 -> SPICLK
- R10 pad 2: 3V3 -> Net-(U2-SPICLK)
- R11 pad 1: EN -> SPIQ
- R11 pad 2: 3V3 -> Net-(U2-SPIQ)
- R12 pad 1: BOOT -> SPID
- R12 pad 2: 3V3 -> Net-(U2-SPID)
- R13 pad 1: Net-(C19-Pad1) -> TX
- R13 pad 2: XTAL_P -> Net-(U2-U0TXD)
- R14 pad 1: DAT2 -> CLK
- R14 pad 2: 3V3 -> Net-(U2-GPIO36)
- R15 pad 1: DAT3 -> SPICS0
- R16 pad 1: CMD -> EN
- R17 pad 1: DAT0 -> BOOT
- R18 pad 1: VBUS -> Net-(C19-Pad1)
- R18 pad 2: Net-(D2-A) -> XTAL_P
- R19 pad 1: DAT1 -> DAT2
- R20 pad 1: IR-OUT -> DAT3
- R20 pad 2: Net-(Q1-B) -> 3V3
- R21 pad 1: Net-(D3-A) -> CMD
- R21 pad 2: VBUS -> 3V3
- R8 pad 1: TX -> SPIHD
- R8 pad 2: Net-(U2-U0TXD) -> Net-(U2-SPIHD)
- R9 pad 1: CLK -> SPIWP
- R9 pad 2: Net-(U2-GPIO36) -> Net-(U2-SPIWP)
- U2 pad 30: SPIHD -> Net-(U2-SPIHD)
- U2 pad 31: SPIWP -> Net-(U2-SPIWP)
- U2 pad 33: SPICLK -> Net-(U2-SPICLK)
- U2 pad 34: SPIQ -> Net-(U2-SPIQ)
- U2 pad 35: SPID -> Net-(U2-SPID)
