File: home.kicad_pcb (KiCad board)
At the start: 6 copper layers, 31.7 x 34.9 mm, 89 parts, among them J1 USB_C_Receptacle_USB2.0_14P, J2 JST, J3 DISPLAY, J4 Micro_SD_Card, J5 VS1838B IR Receiver, Q1 SS8050, SW1 SW_Push, SW2 SW_Push, U1 USBLC6-2SC6, U2 ESP32-S3, U3 SPX3819M5-L-3-3, U4 ESP-PSRAM64H, U5 W25Q128JVSIQ, U6 BH1750FVI-TR, U7 SCD41-D-R2, Y1 40MHz

Commit message: Thurs
Parts:
- removed C20: 100nF, Capacitor_SMD:C_0402_1005Metric
- removed J2: JST, Connector_PinHeader_2.54mm:PinHeader_1x04_P2.54mm_Vertical
- removed REF**: Texas_SWRA117D_2.4GHz_Right, RF_Antenna:Texas_SWRA117D_2.4GHz_Right
- removed TP1, TP2, TP3, TP4, TP5, TP6: TestPoint, TestPoint:TestPoint_Pad_D1.0mm
- removed U7: SCD41-D-R2, Sensor:Sensirion_SCD4x-1EP_10.1x10.1mm_P1.25mm_EP4.8x4.8mm
- added 3V3: TestPoint, TestPoint:TestPoint_Pad_D1.0mm, B.Cu at (153.2, 122.2)
- added GND: TestPoint, TestPoint:TestPoint_Pad_D1.0mm, B.Cu at (151.2, 122.2)
- added RX1: TestPoint, TestPoint:TestPoint_Pad_D1.0mm, B.Cu at (165.1, 97.0)
- added SCL: TestPoint, TestPoint:TestPoint_Pad_D1.0mm, B.Cu at (147.2, 122.2)
- added SDA: TestPoint, TestPoint:TestPoint_Pad_D1.0mm, B.Cu at (149.2, 122.2)
- added TX1: TestPoint, TestPoint:TestPoint_Pad_D1.0mm, B.Cu at (163.1, 97.0)
- C27, C28: moved to B.Cu
- IO45: renamed from TP7; moved to B.Cu
- IO46: renamed from TP8; moved to B.Cu
- R14: moved to F.Cu
- moved C27 73.7 mm to (153.4, 118.7)
- moved C28 73.4 mm to (153.4, 120.0)
- moved R22 56.4 mm to (173.5, 102.4)
- moved R19 54.7 mm to (173.5, 109.3)
- moved R20 52.7 mm to (173.5, 108.2)
- moved R24 52.5 mm to (173.6, 99.7), turned to 90 degrees
- moved R21 50.9 mm to (173.5, 107.0)
- moved G*** 46.2 mm to (149.7, 94.1), turned to -135 degrees
- moved IO46 37.4 mm to (155.9, 102.8), turned to 180 degrees
- moved ANT1 27.0 mm to (141.9, 100.0), turned to 45 degrees
- moved IO45 26.1 mm to (167.1, 97.0), turned to 180 degrees
- moved R23 21.3 mm to (147.1, 122.0), turned to 180 degrees
- moved R26 20.3 mm to (147.1, 120.8), turned to 0 degrees
- moved C22 19.5 mm to (154.1, 102.0), turned to -135 degrees
- moved C24 16.6 mm to (151.5, 101.5), turned to -90 degrees
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- renumbered D2 to K^
Connections:
- J3 pad GND: (no net) -> GND
Routing:
- net EN: track 2.75 -> 37.6 mm, vias 0 -> 3
- net VBUS: track 8.11 -> 38.9 mm
- net Net-(U2-GPIO36): track 28.7 -> 1.37 mm, vias 1 -> 0
- net GND: track 39.4 -> 65.4 mm, vias 51 -> 150
- net BOOT: track 3.29 -> 21.6 mm, vias 1 -> 2
- net IO45: track 0.00 -> 15.5 mm, vias 0 -> 2
- net IR-OUT: track 3.09 -> 18.2 mm, vias 0 -> 2
- net 3V3: track 15.8 -> 29.9 mm, vias 19 -> 28
- net LCD_DC: track 19.6 -> 6.66 mm
- net RX: track 0.00 -> 12.9 mm, vias 0 -> 2
- net CLK: track 1.20 -> 13.6 mm, vias 0 -> 2
- net IR-IN: track 1.29 -> 12.7 mm
- net DAT3: track 26.5 -> 15.5 mm, vias 1 -> 2
- net SCL: track 18.7 -> 29.8 mm, vias 1 -> 6
- net SDA: track 23.5 -> 34.0 mm, vias 3 -> 5
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- added copper zone on In2.Cu, net 3V3
- added copper zone on In1.Cu, net GND
- added copper zone on In3.Cu, net GND
- added copper zone on In4.Cu, net GND
Other:
- board size 31.7 x 34.9 mm -> 33.9 x 35.1 mm
- board text added: "Jonathan Black"
- board text added: "^"
- board text removed: "ESP-32-S3 Lazy Kiwi"
- board text removed: "茉莉花大好き：）"
