File: homequadspi.kicad_pcb (KiCad board)
At the start: 6 copper layers, 33.9 x 35.1 mm, 88 parts, among them J1 USB_C_Receptacle_USB2.0_14P, J2 DISPLAY, J3 Micro_SD_Card, J4 VS1838B IR Receiver, Q1 SS8050, SW1 SW_Push, SW2 SW_Push, U1 USBLC6-2SC6, U2 ESP32-S3, U3 SPX3819M5-L-3-3, U4 ESP-PSRAM64H, U5 W25Q128JVSIQ, U6 MCP9808_DFN, U7 BH1750FVI-TR, Y1 40MHz

Commit message: sklfdjaj
Parts:
- moved C25 22.5 mm to (187.6, 103.9)
- moved R7 20.0 mm to (186.6, 108.6)
- moved C12 15.6 mm to (179.0, 114.0)
- moved C13 15.6 mm to (177.9, 114.0)
- moved R15 14.7 mm to (185.9, 105.1)
- moved U5 1.70 mm to (168.3, 101.1), turned to 0 degrees
- moved U4 1.36 mm to (167.6, 107.7), turned to 90 degrees
Routing:
- net SPICS0: track 22.0 -> 4.99 mm, vias 2 -> 1
- net SPIQ: track 22.2 -> 6.29 mm, vias 0 -> 2
- net VCC_SPI: track 10.7 -> 0.00 mm, vias 4 -> 0
- net SPICS1: track 12.4 -> 2.31 mm
- net GND: track 84.0 -> 76.5 mm, vias 156 -> 141
- net SPICLK: track 12.5 -> 6.32 mm, vias 2 -> 0
- net SPIHD: track 12.6 -> 6.82 mm
- net SPIWP: track 19.3 -> 13.6 mm, vias 2 -> 0
- net SPID: track 11.6 -> 7.61 mm
- net 3V3: track 33.7 -> 32.5 mm, vias 29 -> 27
- removed copper zone on F.Cu, net VCC_SPI
