File: _restore_backup_2026-07-09T23-22-45-189/home.kicad_sch (KiCad schematic)
At the start: 87 parts, among them J1 USB_C_Receptacle_USB2.0_14P, J2 JST, J3 DISPLAY, J4 Micro_SD_Card, J5 VS1838B IR Receiver, Q1 SS8050, SW1 SW_Push, SW2 SW_Push, U1 USBLC6-2SC6, U2 ESP32-S3, U3 SPX3819M5-L-3-3, U4 ESP-PSRAM64H, U5 W25Q128JVSIQ, U6 BH1750FVI-TR, U7 SCD41-D-R2, Y1 40MHz

Commit message: ThursAkiba
Parts:
- removed TP1, TP2, TP3, TP4, TP5, TP6, TP7, TP8: TestPoint, TestPoint:TestPoint_Pad_D1.0mm, symbol Connector:TestPoint
- C1, C16, C21, C4: footprint Capacitor_SMD:C_0402_1005Metric -> Capacitor_SMD:C_0603_1608Metric
- C3: footprint Capacitor_SMD:C_0402_1005Metric -> Capacitor_SMD:C_0201_0603Metric
- L1, L2: footprint Inductor_SMD:L_0402_1005Metric -> Inductor_SMD:L_0603_1608Metric
- R1, R13, R14, R15, R16, R17, R18, R2, R23, R25, R26, R3, R4, R5, R6, R7: footprint Resistor_SMD:R_0402_1005Metric -> Resistor_SMD:R_0603_1608Metric
- R10, R11, R12, R8, R9: footprint Resistor_SMD:R_0201_0603Metric -> Resistor_SMD:R_0402_1005Metric
Connections:
- net 3V3: now also C12.2
- net D+: no longer J1.A6 (D+), J1.B6 (D+), U1.3 (I/O2)
- net D-: no longer J1.A7 (D-), J1.B7 (D-), U1.1 (I/O1)
- net VCC_SPI: no longer C12.2
- new net: J1.A6 (D+), J1.B6 (D+), U1.3 (I/O2)
- new net: J1.A7 (D-), J1.B7 (D-), U1.1 (I/O1)
Other:
- note removed: "GPIO Breakouts"
