File: _restore_backup_2026-07-12T09-39-38-370/home.kicad_pcb (KiCad board)
At the start: 6 copper layers, 31.7 x 34.9 mm, 89 parts, among them J1 USB_C_Receptacle_USB2.0_14P, J2 JST, J3 DISPLAY, J4 Micro_SD_Card, J5 VS1838B IR Receiver, Q1 SS8050, SW1 SW_Push, SW2 SW_Push, U1 USBLC6-2SC6, U2 ESP32-S3, U3 SPX3819M5-L-3-3, U4 ESP-PSRAM64H, U5 W25Q128JVSIQ, U6 BH1750FVI-TR, U7 SCD41-D-R2, Y1 40MHz

Commit message: ThursAkiba
Parts:
- J4: footprint Connector_Card:microSD_HC_Molex_104031-0811 -> parts:MicroSD LCSC
- R14: moved to F.Cu
- moved C29 76.5 mm to (220.4, 133.4), turned to 0 degrees
- moved J5 74.7 mm to (223.8, 129.6), turned to 0 degrees
- moved R14 45.2 mm to (206.8, 135.7), turned to 0 degrees
- moved U7 22.6 mm to (206.8, 91.0)
- moved R25 18.4 mm to (130.2, 98.4), turned to 0 degrees
- moved Q1 16.9 mm to (131.5, 94.6), turned to 0 degrees
- moved D2 16.5 mm to (135.9, 94.9), turned to 0 degrees
- moved R23 13.7 mm to (132.1, 102.4), turned to 0 degrees
- moved R26 12.2 mm to (132.1, 100.9), turned to 0 degrees
- moved D3 11.6 mm to (141.9, 94.9), turned to 0 degrees
- moved J4 6.96 mm to (173.7, 103.5), turned to -90 degrees
- moved C18 3.07 mm to (175.5, 114.8), turned to 90 degrees
- moved C26 0.35 mm to (150.3, 107.9)
- moved REF** 0.09 mm to (152.6, 94.8)
- renumbered R12 to R8-12
Connections:
- J4 pad 9: GND -> (no net)
Routing:
- net Net-(U2-GPIO36): track 28.7 -> 0.00 mm, vias 1 -> 0
- net DAT3: track 26.5 -> 0.00 mm, vias 1 -> 0
- net CMD: track 23.1 -> 0.00 mm, vias 1 -> 0
- net DAT1: track 22.0 -> 0.00 mm, vias 1 -> 0
- net DAT2: track 19.8 -> 0.00 mm, vias 1 -> 0
- net LCD_DC: track 19.6 -> 0.00 mm, vias 1 -> 0
- net DAT0: track 19.4 -> 0.00 mm, vias 1 -> 0
- net SDA: track 23.5 -> 11.1 mm, vias 3 -> 2
- net GND: track 39.4 -> 28.3 mm, vias 51 -> 54
- net LCD_BL: track 8.87 -> 0.00 mm, vias 1 -> 0
- net SCL: track 18.7 -> 13.7 mm, vias 1 -> 0
- net CLK: track 1.20 -> 0.00 mm
- net IR-OUT: track 3.09 -> 1.96 mm
- net TP_INT: track 15.1 -> 14.5 mm
- net FSPICLK: vias 0 -> 1
Other:
- board size 31.7 x 34.9 mm -> 35.5 x 34 mm
- copper layers 6 -> 4
- board text added: "pin 1"
